File: KiCad/MA41_tester_v1/MA-41.kicad_sch (KiCad schematic)
At the start: 0 parts

Commit message: ююю
Changed lines of the file:
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@@
 (kicad_sch (version 20211123) (generator eeschema)
   (paper "A4")
-  (hierarchical_label "GND" (shape input) (at 55.88 78.74 0)
+  (hierarchical_label "GND" (shape input) (at 55.88 104.14 0)
     (effects (font (size 1.27 1.27)) (justify left))
   )
-  (hierarchical_label "UART_TX" (shape bidirectional) (at 55.88 68.58 0)
+  (hierarchical_label "UART_TX" (shape bidirectional) (at 55.88 92.71 0)
     (effects (font (size 1.27 1.27)) (justify left))
   )
-  (hierarchical_label "UART_RX" (shape bidirectional) (at 55.88 63.5 0)
+  (hierarchical_label "UART_RX" (shape bidirectional) (at 55.88 99.06 0)
     (effects (font (size 1.27 1.27)) (justify left))
   )
-  (hierarchical_label "3.3V" (shape output) (at 55.88 83.82 0)
+  (hierarchical_label "NU" (shape bidirectional) (at 55.88 87.63 0)
     (effects (font (size 1.27 1.27)) (justify left))
   )
-  (hierarchical_label "VCC" (shape input) (at 55.88 73.66 0)
+  (hierarchical_label "VCC" (shape input) (at 55.88 81.28 0)
     (effects (font (size 1.27 1.27)) (justify left))
   )
