File: KiCad/MA41_tester_v1/ESP32.kicad_sch (KiCad schematic)
At the start: 0 parts

Commit message: ююю
Changed lines of the file:
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@@
 (kicad_sch (version 20211123) (generator eeschema)
   (paper "A4")
-  (hierarchical_label "GND" (shape bidirectional) (at 45.72 85.09 0)
+  (polyline (pts (xy 83.82 52.07) (xy 45.72 52.07))
+    (stroke (width 0) (type default) (color 0 0 0 0))
+  )
+  (polyline (pts (xy 83.82 97.79) (xy 83.82 52.07))
+    (stroke (width 0) (type default) (color 0 0 0 0))
+  )
+  (polyline (pts (xy 45.72 52.07) (xy 45.72 59.69))
+    (stroke (width 0) (type default) (color 0 0 0 0))
+  )
+  (polyline (pts (xy 45.72 97.79) (xy 83.82 97.79))
+    (stroke (width 0) (type default) (color 0 0 0 0))
+  )
+  (polyline (pts (xy 45.72 59.69) (xy 45.72 97.79))
+    (stroke (width 0) (type default) (color 0 0 0 0))
+  )
+  (hierarchical_label "3(UART0RX)" (shape input) (at 83.82 64.77 180)
+    (effects (font (size 1.27 1.27)) (justify right))
+  )
+  (hierarchical_label "Vin" (shape bidirectional) (at 45.72 93.98 0)
     (effects (font (size 1.27 1.27)) (justify left))
+  )
+  (hierarchical_label "22 SCL" (shape bidirectional) (at 83.82 57.15 180)
+    (effects (font (size 1.27 1.27)) (justify right))
+  )
+  (hierarchical_label "21 SDA" (shape bidirectional) (at 83.82 68.58 180)
+    (effects (font (size 1.27 1.27)) (justify right))
+  )
+  (hierarchical_label "1(UART0TX)" (shape output) (at 83.82 60.96 180)
+    (effects (font (size 1.27 1.27)) (justify right))
+  )
+  (hierarchical_label "18" (shape bidirectional) (at 83.82 86.36 180)
+    (effects (font (size 1.27 1.27)) (justify right))
+  )
+  (hierarchical_label "16(UART2RX)" (shape output) (at 83.82 74.93 180)
+    (effects (font (size 1.27 1.27)) (justify right))
+  )
+  (hierarchical_label "17(UART2TX)" (shape output) (at 83.82 72.39 180)
+    (effects (font (size 1.27 1.27)) (justify right))
+  )
+  (hierarchical_label "GND" (shape bidirectional) (at 45.72 91.44 0)
+    (effects (font (size 1.27 1.27)) (justify left))
+  )
+  (hierarchical_label "19" (shape bidirectional) (at 83.82 83.82 180)
+    (effects (font (size 1.27 1.27)) (justify right))
+  )
+  (hierarchical_label "+3.3V" (shape bidirectional) (at 83.82 93.98 180)
+    (effects (font (size 1.27 1.27)) (justify right))
+  )
+  (hierarchical_label "GND2" (shape bidirectional) (at 83.82 91.44 180)
+    (effects (font (size 1.27 1.27)) (justify right))
   )
   (hierarchical_label "EN" (shape bidirectional) (at 45.72 64.77 0)
     (effects (font (size 1.27 1.27)) (justify left))
   )
+  (hierarchical_label "36(VP)" (shape input) (at 45.72 67.31 0)
+    (effects (font (size 1.27 1.27)) (justify left))
+  )

Commit message: ///
Changed lines of the file:
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@@
     (effects (font (size 1.27 1.27)) (justify right))
+  )
+  (hierarchical_label "32" (shape input) (at 45.72 72.39 0)
+    (effects (font (size 1.27 1.27)) (justify left))
   )
   (hierarchical_label "21 SDA" (shape bidirectional) (at 83.82 68.58 180)
@@
     (effects (font (size 1.27 1.27)) (justify left))
   )
+  (hierarchical_label "33" (shape output) (at 45.72 74.93 0)
+    (effects (font (size 1.27 1.27)) (justify left))
+  )

Commit message: fix com port exception
Changed lines of the file:
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@@
     (stroke (width 0) (type default) (color 0 0 0 0))
-  )
-  (hierarchical_label "3(UART0RX)" (shape input) (at 83.82 64.77 180)
-    (effects (font (size 1.27 1.27)) (justify right))
   )
   (hierarchical_label "Vin" (shape bidirectional) (at 45.72 93.98 0)
@@
     (effects (font (size 1.27 1.27)) (justify right))
   )
-  (hierarchical_label "32" (shape input) (at 45.72 72.39 0)
+  (hierarchical_label "32(Serial1RX)" (shape input) (at 45.72 72.39 0)
     (effects (font (size 1.27 1.27)) (justify left))
   )
@@
     (effects (font (size 1.27 1.27)) (justify right))
   )
-  (hierarchical_label "1(UART0TX)" (shape output) (at 83.82 60.96 180)
-    (effects (font (size 1.27 1.27)) (justify right))
-  )
   (hierarchical_label "18" (shape bidirectional) (at 83.82 86.36 180)
     (effects (font (size 1.27 1.27)) (justify right))
   )
-  (hierarchical_label "16(UART2RX)" (shape output) (at 83.82 74.93 180)
+  (hierarchical_label "16(RX2)" (shape output) (at 83.82 74.93 180)
     (effects (font (size 1.27 1.27)) (justify right))
   )
-  (hierarchical_label "17(UART2TX)" (shape output) (at 83.82 72.39 180)
+  (hierarchical_label "17(TX2)" (shape output) (at 83.82 72.39 180)
     (effects (font (size 1.27 1.27)) (justify right))
   )
@@
     (effects (font (size 1.27 1.27)) (justify left))
   )
-  (hierarchical_label "33" (shape output) (at 45.72 74.93 0)
+  (hierarchical_label "33(Serial1TX)" (shape output) (at 45.72 74.93 0)
     (effects (font (size 1.27 1.27)) (justify left))
   )
